File: Nivara (KiCad)/0mA__10mA_module.kicad_sch (KiCad schematic)
At the start: 7 parts, among them U7 GP8201S-TC50-EW

Commit message: Add files via upload
Parts:
- removed R19, R20, R21: R_0603, PCM_Resistor_SMD_AKL:R_0603_1608Metric, symbol PCM_Resistor_US_AKL:R_0603
Connections:
- net SCLK is gone; now on net +3.3V: U7.1 (SCLK)
- net SDA is gone; now on net +3.3V: U7.2 (SDA)
- net at U7.7 (SEL): now also C5.2, U7.8 (V5V)
Other:
- moved on the sheet: C5, C6, D8, U7

Commit message: Add files via upload
Parts:
- C5, C6: footprint PCM_Capacitor_SMD_AKL:C_0603_1608Metric -> Capacitor_SMD:C_0402_1005Metric
- D10: renamed from D8; footprint PCM_Diode_SMD_AKL:D_SOD-123F -> Diode_SMD:D_SMF
- U7: footprint EastEDA:GP8303-TC50-EW -> External:GP8201S
Other:
- moved on the sheet: C5, C6, D10, U7
