File: Nivara (KiCad)/0v__10v_Module.kicad_sch (KiCad schematic)
At the start: 0 parts

Commit message: Add files via upload
Parts:
- added C2: C_0603, Capacitor_SMD:C_0402_1005Metric, symbol PCM_Capacitor_US_AKL:C_0603
- added D6: MB24F_C7427849, Diode_SMD:Diode_Bridge_Diotec_ABS, symbol EDA:MB24F_C7427849
- added R17, R18: R_0603, Resistor_SMD:R_0603_1608Metric, symbol PCM_Resistor_US_AKL:R_0603
Connections:
- new net: C2.1, D6.1 (-), R17.2
- new net: D6.2 (+), R18.2
- new net 0v_10V: D6.3 (C1)
- new net Ang_0V_10V_IN: C2.2, R17.1, R18.1
- new net GND: D6.4 (C2)
