File: Nivara (KiCad)/0v__32v__module.kicad_sch (KiCad schematic)
At the start: 6 parts, among them U10 LTV-357TB, U9 LTV-357TB

Commit message: Add files via upload
Parts:
- removed R25, R26, R28, R29: R_0603, PCM_Resistor_SMD_AKL:R_0603_1608Metric, symbol PCM_Resistor_US_AKL:R_0603
- removed U10, U9: LTV-357TB, Package_SO:SO-4_4.4x3.6mm_P2.54mm, symbol Isolator:LTV-357T
- added C3: C_0603, Capacitor_SMD:C_0402_1005Metric, symbol PCM_Capacitor_US_AKL:C_0603
- added D7: MB24F_C7427849, Diode_SMD:Diode_Bridge_Diotec_ABS, symbol EDA:MB24F_C7427849
- added R19, R20: R_0603, Resistor_SMD:R_0603_1608Metric, symbol PCM_Resistor_US_AKL:R_0603
Connections:
- net GND: now also D7.4 (C2)
- new net: C3.1, D7.1 (-), R19.2
- new net: D7.2 (+), R20.2
- new net 0V_32V: D7.3 (C1)
- new net Analog_0-32_IN1: C3.2, R19.1, R20.1
