File: Nivara (KiCad)/Digit_module.kicad_sch (KiCad schematic)
At the start: 8 parts

Commit message: Add files via upload
Other:
- moved on the sheet: D6, D7, OC5, OC6, R15, R16, R17, R18

Commit message: Add files via upload
Parts:
- OC5, OC6: footprint PCM_Package_SO_AKL:SO-4_4.4x3.9mm_P2.54mm -> Package_SO:SO-4_4.4x2.3mm_P1.27mm
- R22: renamed from R15; footprint PCM_Resistor_SMD_AKL:R_0603_1608Metric -> Resistor_SMD:R_0603_1608Metric
- R23: renamed from R16; footprint PCM_Resistor_SMD_AKL:R_0603_1608Metric -> Resistor_SMD:R_0603_1608Metric
- R24: renamed from R17; footprint PCM_Resistor_SMD_AKL:R_0603_1608Metric -> Resistor_SMD:R_0603_1608Metric
- R25: renamed from R18; footprint PCM_Resistor_SMD_AKL:R_0603_1608Metric -> Resistor_SMD:R_0603_1608Metric
- renumbered D6 to D8, D7 to D9
Other:
- moved on the sheet: D8, D9, OC5, OC6, R22, R23, R24, R25
