File: Nivara (KiCad)/Input_NPN.kicad_sch (KiCad schematic)
At the start: 8 parts

Commit message: Add files via upload
Parts:
- OC1, OC2: footprint PCM_Package_SO_AKL:SO-4_4.4x3.9mm_P2.54mm -> Package_SO:SO-4_4.4x2.3mm_P1.27mm
- R5: renamed from R2; footprint PCM_Resistor_SMD_AKL:R_0603_1608Metric -> Resistor_SMD:R_0603_1608Metric
- R6: renamed from R3; footprint PCM_Resistor_SMD_AKL:R_0603_1608Metric -> Resistor_SMD:R_0603_1608Metric
- R7: renamed from R4; footprint PCM_Resistor_SMD_AKL:R_0603_1608Metric -> Resistor_SMD:R_0603_1608Metric
- R8: renamed from R5; footprint PCM_Resistor_SMD_AKL:R_0603_1608Metric -> Resistor_SMD:R_0603_1608Metric
Other:
- moved on the sheet: D2, D3, OC1, OC2, R5, R6, R7, R8
