File: Nivara (KiCad)/Nivara.kicad_pcb (KiCad board)
At the start: 2 copper layers, 87 parts, among them J1 Terminal_2, J10 Terminal_6, J2 Terminal_2, J3 Terminal_4, J4 Terminal_4, J5 Terminal_2, J6 Terminal_2, J7 Terminal_3, J8 Terminal_3, J9 Terminal_4, U1 ESP32-S3-WROOM-1, U1 GAQY211G2S, U2 GAQY211G2S, U4 AP63203WU, U7 GP8201S-TC50-EW, U8 GP8303-TC50-EW

Commit message: Add files via upload
Parts:
- removed OC3: LTV-357T-B, PCM_Package_SO_AKL:SO-4_4.4x3.9mm_P2.54mm
- moved U2 79.5 mm to (279.6, 221.8), turned to 180 degrees
- moved D7 68.0 mm to (253.7, 169.0), turned to -90 degrees
- moved D3 61.4 mm to (258.7, 169.0), turned to -90 degrees
- moved R25 61.2 mm to (257.0, 208.7), turned to -90 degrees
- moved C1 60.3 mm to (255.7, 193.7), turned to 90 degrees
- moved TP4 58.9 mm to (258.9, 188.1), turned to 90 degrees
- moved R1 57.8 mm to (257.5, 193.7), turned to -90 degrees
- moved D2 57.5 mm to (261.8, 169.0), turned to -90 degrees
- moved C2 55.1 mm to (266.3, 173.6), turned to 180 degrees
- moved R29 53.4 mm to (261.4, 213.4), turned to 90 degrees
- moved R9 52.5 mm to (254.0, 180.3), turned to -90 degrees
- moved R11 51.5 mm to (255.3, 184.2), turned to -90 degrees
- moved C10 50.8 mm to (267.8, 170.3), turned to 90 degrees
- moved D8 50.0 mm to (281.5, 182.8), turned to 180 degrees
- moved R13 49.7 mm to (255.3, 174.4), turned to -90 degrees
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
Commit message: Add files via upload
Parts:
- removed C10, C11, C12, C18, C8, C9: C_0603, PCM_Capacitor_SMD_AKL:C_0603_1608Metric
- removed the C2 at (279.4, 213.6)
- removed the C2 at (266.3, 173.6)
- removed the D3 at (258.7, 169.0)
- removed the D3 at (260.5, 207.2)
- removed the D4 at (254.3, 142.1)
- removed the D4 at (275.8, 213.7)
- removed the D6 at (252.8, 190.7)
- removed the D6 at (292.2, 170.3)
- removed the D8 at (260.5, 199.4)
- removed the D8 at (281.5, 182.8)
- removed JP1: SolderJumper_2_Open, Jumper:SolderJumper-2_P1.3mm_Open_RoundedPad1.0x1.5mm
- removed L1: L_Iron, Inductor_SMD:L_Bourns-SRN6028
- removed the OC4 at (280.9, 154.6)
- removed the OC4 at (268.3, 154.2)
- removed the OC5 at (275.1, 154.5)
- removed the OC5 at (254.7, 153.8)
- removed the R10 at (271.8, 213.4)
- removed the R10 at (268.4, 202.3)
- removed the R12 at (264.6, 203.6)
- removed the R12 at (285.9, 201.2)
- removed the R13 at (255.3, 174.4)
- removed the R13 at (288.4, 194.1)
- removed the R16 at (274.1, 200.9)
- removed the R16 at (271.0, 180.5)
- removed R29, R50, R51: R_0603, PCM_Resistor_SMD_AKL:R_0603_1608Metric
- removed the R6 at (274.3, 194.1)
- removed the R6 at (277.9, 164.8)
- removed the R9 at (267.5, 164.4)
- removed the R9 at (254.0, 180.3)
- removed TP1, TP2, TP3, TP4: TestPoint, TestPoint:TestPoint_Keystone_5015_Micro_Mini
- removed the U1 at (286.8, 154.7)
- removed the U1 at (280.0, 119.7)
- added C2: C_0603, Capacitor_SMD:C_0402_1005Metric, F.Cu at (240.7, 79.6)
- added D10: SMF24A, Diode_SMD:D_SMF, F.Cu at (287.2, 69.1)
- added D3: DL4007, Diode_SMD:D_0805_2012Metric_Pad1.15x1.40mm_HandSolder, F.Cu at (225.8, 84.7)
- added D4: DL4007, Diode_SMD:D_0805_2012Metric_Pad1.15x1.40mm_HandSolder, F.Cu at (250.4, 100.6)
- added D6: MB24F_C7427849, Diode_SMD:Diode_Bridge_Diotec_ABS, F.Cu at (239.6, 75.3)
- added D8: DL4007, Diode_SMD:D_0805_2012Metric_Pad1.15x1.40mm_HandSolder, F.Cu at (234.5, 100.6)
- added D9: DL4007, Diode_SMD:D_0805_2012Metric_Pad1.15x1.40mm_HandSolder, F.Cu at (234.5, 103.6)
- added K1: G2RL-1, Relay_THT:Relay_SPDT_Omron_G2RL-1, F.Cu at (191.5, 96.8)
- added K2: G2RL-1, Relay_THT:Relay_SPDT_Omron_G2RL-1, F.Cu at (191.5, 82.7)
- added OC2: LTV-357T-B, Package_SO:SO-4_4.4x2.3mm_P1.27mm, F.Cu at (228.3, 78.1)
- added OC3: LTV-357T-B, Package_SO:SO-4_4.4x2.3mm_P1.27mm, F.Cu at (252.9, 93.0)
- added OC4: LTV-357T-B, Package_SO:SO-4_4.4x2.3mm_P1.27mm, F.Cu at (252.9, 97.1)
- added OC5: LTV-357T-B, Package_SO:SO-4_4.4x2.3mm_P1.27mm, F.Cu at (237.0, 93.0)
- added OC6: LTV-357T-B, Package_SO:SO-4_4.4x2.3mm_P1.27mm, F.Cu at (237.0, 97.1)
- added Q1: ~, Button_Switch_THT:SW_NKK_G1xJP, F.Cu at (190.9, 64.4)
- added R10: R_0603, Resistor_SMD:R_0603_1608Metric, F.Cu at (245.9, 94.6)
- added R12: R_0603, Resistor_SMD:R_0603_1608Metric, F.Cu at (245.9, 99.6)
- added R13: R_0603, Resistor_SMD:R_0603_1608Metric, F.Cu at (257.5, 77.7)
- added R16: R_0603, Resistor_SMD:R_0603_1608Metric, F.Cu at (257.5, 83.7)
- added R18: R_0603, Resistor_SMD:R_0603_1608Metric, F.Cu at (237.2, 82.4)
- added R26: R_0603, Resistor_SMD:R_0603_1608Metric, F.Cu at (219.0, 112.3)
- added R27: R_0603, Resistor_SMD:R_0603_1608Metric, F.Cu at (215.5, 112.3)
- added R28: R_0603, Resistor_SMD:R_0603_1608Metric, F.Cu at (212.5, 102.7)
- added R4: R_0603, Resistor_SMD:R_0603_1608Metric, F.Cu at (277.8, 75.9)
- added R5: R_0603, Resistor_SMD:R_0603_1608Metric, F.Cu at (221.4, 73.1)
- added R6: R_0603, Resistor_SMD:R_0603_1608Metric, F.Cu at (221.4, 75.7)
- added R9: R_0603, Resistor_SMD:R_0603_1608Metric, F.Cu at (245.9, 92.1)
- added U1: ESP32-S3-WROOM-1, RF_Module:ESP32-S3-WROOM-1, F.Cu at (276.8, 102.9)
- added U3: GAQY211G2S, Package_SO:SOP-4_3.8x4.1mm_P2.54mm, F.Cu at (242.5, 63.3)
- added U5: GAQY211G2S, Package_SO:SOP-4_3.8x4.1mm_P2.54mm, F.Cu at (227.0, 63.3)
- added U6: GAQY211G2S, Package_SO:SOP-4_3.8x4.1mm_P2.54mm, F.Cu at (219.5, 63.3)
- C1, C3, C4, C5, C6, C7: footprint PCM_Capacitor_SMD_AKL:C_0603_1608Metric -> Capacitor_SMD:C_0402_1005Metric
- D1: value SM712 -> SM712_SOT23; footprint PCM_Package_TO_SOT_SMD_AKL:SOT-23 -> Package_TO_SOT_SMD:SOT-23_Handsoldering
- D7: value DL4007 -> MB24F_C7427849; footprint Diode_SMD:D_0805_2012Metric_Pad1.15x1.40mm_HandSolder -> Diode_SMD:Diode_Bridge_Diotec_ABS
- J1, J2, J5, J6: value Terminal_2 -> Screw_Terminal_2_P5.00mm
- J10: value Terminal_6 -> Screw_Terminal_6_P5.00mm
- J3, J4, J9: value Terminal_4 -> Screw_Terminal_4_P5.00mm
- J7, J8: value Terminal_3 -> Screw_Terminal_3_P5.00mm
- OC1: footprint PCM_Package_SO_AKL:SO-4_4.4x3.9mm_P2.54mm -> Package_SO:SO-4_4.4x2.3mm_P1.27mm
- R1, R11, R14, R15, R17, R19, R2, R20, R21, R22, R23, R24, R25, R3, R7, R8: footprint PCM_Resistor_SMD_AKL:R_0603_1608Metric -> Resistor_SMD:R_0603_1608Metric
- U2: value GAQY211G2S -> ~; footprint EastEDA:GAQY211G2s -> External:RSM3485ECHT
- U4: value AP63203WU -> GAQY211G2S; footprint Package_TO_SOT_SMD:TSOT-23-6 -> Package_SO:SOP-4_3.8x4.1mm_P2.54mm
- U7: footprint EastEDA:GP8303-TC50-EW -> External:GP8201S
- U8: footprint EastEDA:ESOP-10_L4.9-W3.9-P1.00-LS6.1-BL-EP -> External:GP8303
- moved U2 152.2 mm to (249.5, 72.6), turned to 90 degrees
- moved C5 145.1 mm to (196.5, 67.8), turned to 90 degrees
- moved C6 141.1 mm to (193.5, 67.9), turned to 90 degrees
- moved D1 137.5 mm to (279.0, 69.9), turned to 0 degrees
- moved C1 136.9 mm to (272.5, 57.8)
- moved R1 136.1 mm to (276.0, 58.8), turned to 90 degrees
- moved C4 123.8 mm to (285.7, 76.2), turned to 0 degrees
- moved C7 122.1 mm to (206.0, 106.3), turned to 90 degrees
- moved R14 122.0 mm to (254.5, 77.7), turned to 90 degrees
- moved R15 120.9 mm to (254.5, 83.7), turned to 90 degrees
- moved U4 117.6 mm to (234.5, 63.3), turned to 90 degrees
- moved R2 112.6 mm to (269.0, 58.7), turned to 90 degrees
- moved R24 112.4 mm to (230.1, 97.1)
- moved R25 112.4 mm to (230.1, 99.6), turned to 0 degrees
- moved R23 112.2 mm to (230.1, 94.6)
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Connections:
- net /Board/RS485-A renamed /RS485-A
- net /Board/RS485-B renamed /RS485-B
- C3 pad 1: Net-(U4-SW) -> Net-(D7--)
- C3 pad 2: Net-(U4-BST) -> /Board/0v_32v/Analog_0-32_IN1
- C4 pad 2: /Board/4_20mA/A_4mA_20mA_Out -> /Board/Analog_4-20_IN1
- C5 pad 2: Net-(U7-V5V) -> Net-(U7-SEL)
- D1 pad 1: GND -> /Board/RS485_B
- D1 pad 2: +3.3V -> /Board/RS485_A
- D7 pad 1: Net-(D7-K) -> Net-(D7--)
- D7 pad 2: GND -> Net-(D7-+)
- OC1 pad 1: Net-(D3-K) -> Net-(D2-K)
- OC1 pad 4: /Board_NIVARA/Input_NPN/NPN-Digit_input_1 -> /Board/Input_NPN/NPN-Digit_IN1
- R1 pad 2: Net-(U1-EN) -> /Board/Start | Stop
- R11 pad 1: /Board_NIVARA/0v__10v_Module/D_0v__10v -> /Board/PNP_IN2
- R11 pad 2: Net-(D4--) -> Net-(D5-K)
- R14 pad 1: /Board/4_20mA/A_4mA_20mA_Out -> /Board/Output_NPN/NPN_IN1
- R14 pad 2: GND -> Net-(R14-Pad2)
- R15 pad 1: /Board/Digit_module/Plu_Dig_IN1 -> /Board/Output_PNP/PNP_input_0
- R17 pad 1: +3.3V -> /Board/Analog_0_10_IN1
- R17 pad 2: /Board_NIVARA/Input_NPN/NPN-Digit_input_2 -> Net-(D6--)
- R19 pad 1: /Board/0_10mA/SCLK -> /Board/0v_32v/Analog_0-32_IN1
- R19 pad 2: +3.3V -> Net-(D7--)
- R2 pad 1: Net-(JP1-A) -> +3.3V
- R2 pad 2: Net-(U4-FB) -> Net-(U1-EN)
- R20 pad 1: /Board/0_10mA/SDA -> /Board/0v_32v/Analog_0-32_IN1
- R20 pad 2: +3.3V -> Net-(D7-+)
- R21 pad 1: Net-(U7-SEL) -> /Board/Analog_4-20_IN1
- R21 pad 2: Net-(U7-V5V) -> GND
- R22 pad 1: /Board/0_10mA/SDA -> /Board/Digit_module/Plu_Dig_IN1
- R22 pad 2: +3.3V -> Net-(D8-K)
- R23 pad 1: /Board/0_10mA/SCLK -> +3.3V
- R23 pad 2: +3.3V -> /Board/Digit_module/Plu_Digit_IN1
- R24 pad 1: GND -> /Board/Digit_module/Plu_Dig_IN2
- R24 pad 2: Net-(U8-SET) -> Net-(D9-K)
- R25 pad 2: /Board_NIVARA/RUN/STOP -> /Board/Digit_module/Plu_Digit_IN2
- R3 pad 1: Net-(U4-FB) -> Net-(U2-B)
- R3 pad 2: GND -> /Board/RS485_A
- R7 pad 1: /Board/Input_PNP/PNP_in_2 -> /Board/NPN_IN2
- R7 pad 2: Net-(D5-K) -> Net-(D3-K)
- R8 pad 1: /Board/Input_PNP/PNP_Digit_1 -> +3.3V
- R8 pad 2: GND -> /Board/Input_NPN/NPN-Digit_IN2
- REF** pad 1: (no net) -> GND (x2)
- U2 pad 1: Net-(R10-Pad2) -> +3.3V
- U2 pad 3: GND -> /Board/RS485/UART_OUT
- U2 pad 4: /Board/NPN_OUT1 -> /Board/RS485/UART_IN
- U4 pad 1: Net-(U4-FB) -> Net-(R14-Pad2)
- U4 pad 2: VCC -> GND
- U4 pad 3: VCC -> GND
- U4 pad 4: GND -> /Board/Output_NPN/NPN_OUT2
- U7 pad 1: /Board/0_10mA/SCLK -> +3.3V
- U7 pad 2: /Board/0_10mA/SDA -> +3.3V
- U7 pad 8: Net-(U7-V5V) -> Net-(U7-SEL)
- U8 pad 1: /Board/0_10mA/SCLK -> +3.3V
- U8 pad 2: /Board/0_10mA/SDA -> +3.3V
Routing:
- net GND: track 0.00 -> 356.2 mm, vias 0 -> 10
- net +3.3V: track 0.00 -> 218.9 mm, vias 0 -> 4
- net /Board/RLY1/RLY_Enable_2: track 0.00 -> 124.1 mm, vias 0 -> 2
- net /Board/0_10mA/Ang_Out: track 0.00 -> 114.9 mm, vias 0 -> 2
- net /Board/Start | Stop: track 0.00 -> 114.7 mm, vias 0 -> 2
- net VCC: track 0.00 -> 101.4 mm, vias 0 -> 1
- net /Board/Analog_4-20_IN1: track 0.00 -> 94.0 mm, vias 0 -> 1
- net /Board/RLY_2_COM: track 0.00 -> 92.5 mm
- net /Board/RLY1/RLY_Enable_1: track 0.00 -> 81.9 mm, vias 0 -> 1
- net /Board/RLY_2_NC: track 0.00 -> 68.5 mm
- net /Board/PNP_IN2: track 0.00 -> 67.2 mm, vias 0 -> 1
- net Net-(U1-EN): track 0.00 -> 67.0 mm, vias 0 -> 2
- net /Board/PNP_IN1: track 0.00 -> 66.7 mm, vias 0 -> 1
- net /Board/Output_NPN/NPN_IN0: track 0.00 -> 55.1 mm, vias 0 -> 2
- net /Board/Output_NPN/NPN_IN1: track 0.00 -> 52.4 mm, vias 0 -> 2
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- added copper zone on B.Cu, net (none)
- added copper zone on F.Cu, net (none)
- added copper zone on In1.Cu, net GND
- added copper zone on In2.Cu, net VCC
Other:
- copper layers 2 -> 4
