File: Nivara (KiCad)/Nivara.kicad_sch (KiCad schematic)
At the start: 11 parts, among them J1 Screw_Terminal_2_P5.00mm, J10 Screw_Terminal_6_P5.00mm, J2 Screw_Terminal_2_P5.00mm, J3 Screw_Terminal_4_P5.00mm, J4 Screw_Terminal_4_P5.00mm, J5 Screw_Terminal_2_P5.00mm, J6 Screw_Terminal_2_P5.00mm, J7 Screw_Terminal_3_P5.00mm, J8 Screw_Terminal_3_P5.00mm, J9 Screw_Terminal_4_P5.00mm

Commit message: Add files via upload
Connections:
- net Board/RLY_1_NO is gone; now on net Board/RLY_1_NO: J10.4
- net Board/RLY_1_NO: no longer J10.3
- new net Board/RLY_1_NO: J10.3
Other:
- moved on the sheet: J1, J10, J2, J3, J4, J5, J6, J7, J8, J9
