File: Nivara (KiCad)/OUT__4__20.kicad_sch (KiCad schematic)
At the start: 5 parts, among them U8 GP8303-TC50-EW

Commit message: Add files via upload
Other:
- moved on the sheet: C7, R22, R23, R24

Commit message: Add files via upload
Parts:
- C7: footprint PCM_Capacitor_SMD_AKL:C_0603_1608Metric -> Capacitor_SMD:C_0402_1005Metric
- R26: renamed from R22; footprint PCM_Resistor_SMD_AKL:R_0603_1608Metric -> Resistor_SMD:R_0603_1608Metric
- R27: renamed from R23; footprint PCM_Resistor_SMD_AKL:R_0603_1608Metric -> Resistor_SMD:R_0603_1608Metric
- R28: renamed from R24; footprint PCM_Resistor_SMD_AKL:R_0603_1608Metric -> Resistor_SMD:R_0603_1608Metric
- U8: footprint EastEDA:ESOP-10_L4.9-W3.9-P1.00-LS6.1-BL-EP -> External:GP8303
Other:
- moved on the sheet: C7, R26, R27, R28
