File: Nivara (KiCad)/Output_NPN.kicad_sch (KiCad schematic)
At the start: 4 parts, among them U2 GAQY211G2S, U3 GAQY211G2S

Commit message: Add files via upload
Parts:
- R13: renamed from R10; footprint PCM_Resistor_SMD_AKL:R_0603_1608Metric -> Resistor_SMD:R_0603_1608Metric
- R14: renamed from R11; footprint PCM_Resistor_SMD_AKL:R_0603_1608Metric -> Resistor_SMD:R_0603_1608Metric
- U3: renamed from U2; footprint EastEDA:GAQY211G2s -> Package_SO:SOP-4_3.8x4.1mm_P2.54mm
- U4: renamed from U3; footprint EastEDA:GAQY211G2s -> Package_SO:SOP-4_3.8x4.1mm_P2.54mm
Connections:
- net NPN_OUT0 is gone; now on net NPN_OUT1: U3.4
- net NPN_OUT1: no longer U4.4
- new net NPN_OUT2: U4.4
Other:
- moved on the sheet: U3, U4
