File: Nivara (KiCad)/Output_PNP.kicad_sch (KiCad schematic)
At the start: 4 parts, among them U3 GAQY211G2S, U4 GAQY211G2S

Commit message: Add files via upload
Parts:
- R15: renamed from R12; footprint PCM_Resistor_SMD_AKL:R_0603_1608Metric -> Resistor_SMD:R_0603_1608Metric
- R16: renamed from R13; footprint PCM_Resistor_SMD_AKL:R_0603_1608Metric -> Resistor_SMD:R_0603_1608Metric
- U5: renamed from U3; footprint EastEDA:GAQY211G2s -> Package_SO:SOP-4_3.8x4.1mm_P2.54mm
- U6: renamed from U4; footprint EastEDA:GAQY211G2s -> Package_SO:SOP-4_3.8x4.1mm_P2.54mm
Changed lines of the file:
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@@
-	(wire
-		(pts
-			(xy 137.16 140.97) (xy 137.16 144.78)
-		)
-		(stroke
-			(width 0)
-			(type default)
-		)
-	)
-	(wire
-		(pts
-			(xy 172.72 129.54) (xy 172.72 132.08)
-		)
-		(stroke
-			(width 0)
-			(type default)
-		)
-	)
 	(wire
 		(pts
@@
 		(dnp no)
 		(fields_autoplaced yes)
-		(property "Reference" "U3"
+		(property "Reference" "U5"
 			(at 153.67 118.11 0)
 			(effects
@@
 			)
 		)
-		(property "Footprint" "EastEDA:GAQY211G2s"
+		(property "Footprint" "Package_SO:SOP-4_3.8x4.1mm_P2.54mm"
 			(at 152.4 148.59 0)
 			(effects
@@
 			(project ""
 				(path "/42622735-4343-4315-af64-a45701a752b6/711b914f-41ac-411e-bef3-8ade05c9a19b/8cb3855c-1036-4639-b2fc-e41c31887560"
-					(reference "U3")
+					(reference "U5")
 					(unit 1)
 				)
@@
 		(dnp no)
 		(fields_autoplaced yes)
-		(property "Reference" "#PWR028"
+		(property "Reference" "#PWR027"
 			(at 205.74 113.03 0)
 			(effects
@@
 			(project ""
 				(path "/42622735-4343-4315-af64-a45701a752b6/711b914f-41ac-411e-bef3-8ade05c9a19b/8cb3855c-1036-4639-b2fc-e41c31887560"
-					(reference "#PWR028")
+					(reference "#PWR027")
 					(unit 1)
 				)
@@
 		(on_board yes)
 		(dnp no)
-		(property "Reference" "R12"
+		(property "Reference" "R15"
 			(at 132.588 121.158 90)
 			(effects
@@
 			)
 		)
-		(property "Footprint" "PCM_Resistor_SMD_AKL:R_0603_1608Metric"
+		(property "Footprint" "Resistor_SMD:R_0603_1608Metric"
 			(at 142.24 125.73 0)
 			(effects
@@
 			(project "Nivara Controls"
 				(path "/42622735-4343-4315-af64-a45701a752b6/711b914f-41ac-411e-bef3-8ade05c9a19b/8cb3855c-1036-4639-b2fc-e41c31887560"
-					(reference "R12")
+					(reference "R15")
 					(unit 1)
 				)
@@
 	(symbol
 		(lib_id "power:GND")
-		(at 137.16 144.78 270)
+		(at 137.16 140.97 270)
 		(unit 1)
 		(exclude_from_sim no)
@@
 		(dnp no)
 		(fields_autoplaced yes)
-		(property "Reference" "#PWR026"
-			(at 130.81 144.78 0)
+		(property "Reference" "#PWR024"
+			(at 130.81 140.97 0)
 			(effects
 				(font
@@
 		)
 		(property "Value" "GND"
-			(at 133.35 144.7799 90)
+			(at 133.35 140.9699 90)
 			(effects
 				(font
@@
 		)
 		(property "Footprint" ""
-			(at 137.16 144.78 0)
+			(at 137.16 140.97 0)
 			(effects
 				(font
@@
 		)
 		(property "Datasheet" ""
-			(at 137.16 144.78 0)
+			(at 137.16 140.97 0)
 			(effects
 				(font
@@
 		)
 		(property "Description" "Power symbol creates a global label with name \"GND\" , ground"
-			(at 137.16 144.78 0)
+			(at 137.16 140.97 0)
 			(effects
 				(font
@@
 			(project ""
 				(path "/42622735-4343-4315-af64-a45701a752b6/711b914f-41ac-411e-bef3-8ade05c9a19b/8cb3855c-1036-4639-b2fc-e41c31887560"
-					(reference "#PWR026")
+					(reference "#PWR024")
 					(unit 1)
 				)
@@
 		(dnp no)
 		(fields_autoplaced yes)
-		(property "Reference" "#PWR027"
+		(property "Reference" "#PWR025"
 			(at 168.91 127 0)
 			(effects
@@
 			(project ""
 				(path "/42622735-4343-4315-af64-a45701a752b6/711b914f-41ac-411e-bef3-8ade05c9a19b/8cb3855c-1036-4639-b2fc-e41c31887560"
-					(reference "#PWR027")
+					(reference "#PWR025")
 					(unit 1)
 				)
@@
 	(symbol
 		(lib_id "power:GND")
-		(at 172.72 132.08 0)
-		(unit 1)
-		(exclude_from_sim no)
-		(in_bom yes)
-		(on_board yes)
-		(dnp no)
-		(property "Reference" "#PWR025"
-			(at 172.72 138.43 0)
+		(at 172.72 129.54 270)
+		(unit 1)
+		(exclude_from_sim no)
+		(in_bom yes)
+		(on_board yes)
+		(dnp no)
+		(property "Reference" "#PWR026"
+			(at 166.37 129.54 0)
 			(effects
 				(font
@@
 		)
 		(property "Value" "GND"
-			(at 172.72 136.398 0)
+			(at 168.402 129.54 0)
 			(effects
 				(font
@@
 		)
 		(property "Footprint" ""
-			(at 172.72 132.08 0)
+			(at 172.72 129.54 0)
 			(effects
 				(font
@@
 		)
 		(property "Datasheet" ""
-			(at 172.72 132.08 0)
+			(at 172.72 129.54 0)
 			(effects
 				(font
@@
 		)
 		(property "Description" "Power symbol creates a global label with name \"GND\" , ground"
-			(at 172.72 132.08 0)
+			(at 172.72 129.54 0)
 			(effects
 				(font
@@
 			(project "Nivara Controls"
 				(path "/42622735-4343-4315-af64-a45701a752b6/711b914f-41ac-411e-bef3-8ade05c9a19b/8cb3855c-1036-4639-b2fc-e41c31887560"
-					(reference "#PWR025")
+					(reference "#PWR026")
 					(unit 1)
 				)
@@
 		(dnp no)
 		(fields_autoplaced yes)
-		(property "Reference" "U4"
+		(property "Reference" "U6"
 			(at 189.23 106.68 0)
 			(effects
@@
 			)
 		)
-		(property "Footprint" "EastEDA:GAQY211G2s"
+		(property "Footprint" "Package_SO:SOP-4_3.8x4.1mm_P2.54mm"
 			(at 187.96 137.16 0)
 			(effects
@@
 			(project "Nivara Controls"
 				(path "/42622735-4343-4315-af64-a45701a752b6/711b914f-41ac-411e-bef3-8ade05c9a19b/8cb3855c-1036-4639-b2fc-e41c31887560"
-					(reference "U4")
+					(reference "U6")
 					(unit 1)
 				)
@@
 		(on_board yes)
 		(dnp no)
-		(property "Reference" "R13"
+		(property "Reference" "R16"
 			(at 169.418 109.728 90)
 			(effects
@@
 			)
 		)
-		(property "Footprint" "PCM_Resistor_SMD_AKL:R_0603_1608Metric"
+		(property "Footprint" "Resistor_SMD:R_0603_1608Metric"
 			(at 179.07 114.3 0)
 			(effects
@@
 			(project "Nivara Controls"
 				(path "/42622735-4343-4315-af64-a45701a752b6/711b914f-41ac-411e-bef3-8ade05c9a19b/8cb3855c-1036-4639-b2fc-e41c31887560"
-					(reference "R13")
-					(unit 1)
-				)
+					(reference "R16")
+					(unit 1)
+				)
