File: Nivara (KiCad)/Placa_Nivara.kicad_sch (KiCad schematic)
At the start: 3 parts, among them U1 ESP32-S3-WROOM-1

Commit message: Add files via upload
Parts:
- added R1: R_0603, Resistor_SMD:R_0603_1608Metric, symbol PCM_Resistor_US_AKL:R_0603
- C1: footprint PCM_Capacitor_SMD_AKL:C_0603_1608Metric -> Capacitor_SMD:C_0402_1005Metric
- R2: renamed from R1; footprint PCM_Resistor_SMD_AKL:R_0603_1608Metric -> Resistor_SMD:R_0603_1608Metric
- U1: footprint ESP32-S3-WROM-1:ESP32-S3-WROOM-1 -> RF_Module:ESP32-S3-WROOM-1
Connections:
- net +3.3V: now also R1.1
- net Start | Stop: now also R1.2
Other:
- sheet RS485 ports: added RS485_A, RS485_B; removed RS485-A, RS485-B
- moved on the sheet: C1, R2
