File: Nivara (KiCad)/RLY_MODULE_1.kicad_sch (KiCad schematic)
At the start: 3 parts, among them K3 G2RL-1, K4 G2RL-1

Commit message: Add files via upload
Parts:
- Q1: renamed from Q2; footprint (none) -> Button_Switch_THT:SW_NKK_G1xJP
- renumbered K3 to K1, K4 to K2
Connections:
- net ON_RLY_1 renamed RLY_Enable_1
- net ON_RLY_2 renamed RLY_Enable_2
Other:
- moved on the sheet: K1, K2, Q1
